File: kicad_pami/pami_2026/pami_2026.kicad_pcb (KiCad board)
At the start: 4 copper layers, 50 x 80 mm, 69 parts, among them J1 Conn_01x04_Socket, J10 Conn_01x07_Socket, J11 Conn_01x06, J12 Conn_01x06, J14 Conn_01x03_Pin, J2 Conn_01x03_Pin, J3 Conn_01x04_Pin, J4 Conn_01x02_Pin, J5 Conn_01x05_Pin, J7 Conn_01x03_Pin, J8 USB_C_Receptacle_USB2.0_14P, J9 Conn_01x04_Pin, Q1 NMOS, Q2 NMOS, Q3 NMOS, SW1 SW_Push, SW2 SW_DIP_x01, SW3 SW_Push_Open, SW4 SW_Reed, SW5 SW_Push, SW6 SW_Push, U1 DRV8833RTY, U2 ESP32-S3-MINI-1, U3 LD1117S33TR_SOT223, U4 L7805

Commit message: fin PCB
Parts:
- added J6: Conn_01x02_Pin, Connector_JST:JST_XH_B2B-XH-A_1x02_P2.50mm_Vertical, F.Cu at (59.9, 108.5)
- added REF**: OSHW-Logo2_7.3x6mm_SilkScreen, Symbol:OSHW-Logo2_7.3x6mm_SilkScreen, B.Cu at (48.8, 113.0)
- added kibuzzard-68DE307B: G***, kibuzzard-68DE307B, F.Cu at (81.0, 97.3)
- added kibuzzard-68DE308C: G***, kibuzzard-68DE308C, F.Cu at (51.2, 97.3)
- added kibuzzard-68DE30BC: G***, kibuzzard-68DE30BC, F.Cu at (67.3, 83.7)
- added kibuzzard-68DE30BC: G***, kibuzzard-68DE30BC, B.Cu at (64.5, 84.1)
- added kibuzzard-68DE30D9: G***, kibuzzard-68DE30D9, F.Cu at (65.9, 76.3)
- added kibuzzard-68DE30FA: G***, kibuzzard-68DE30FA, F.Cu at (79.1, 105.9)
- added kibuzzard-68DE3110: G***, kibuzzard-68DE3110, F.Cu at (52.8, 105.9)
- added kibuzzard-68DE3123: G***, kibuzzard-68DE3123, F.Cu at (48.3, 113.5)
- added kibuzzard-68DE313B: G***, kibuzzard-68DE313B, F.Cu at (83.8, 113.5)
- added kibuzzard-68DE3201: G***, kibuzzard-68DE3201, F.Cu at (68.7, 53.0)
- added kibuzzard-68DE3215: G***, kibuzzard-68DE3215, F.Cu at (59.3, 45.5)
- added kibuzzard-68DE323F: G***, kibuzzard-68DE323F, F.Cu at (43.4, 94.7)
- added kibuzzard-68DE324D: G***, kibuzzard-68DE324D, F.Cu at (50.4, 90.2)
- added kibuzzard-68DE325B: G***, kibuzzard-68DE325B, F.Cu at (51.2, 86.2)
- added kibuzzard-68DE326F: G***, kibuzzard-68DE326F, F.Cu at (51.6, 81.8)
- added kibuzzard-68DE32D9: G***, kibuzzard-68DE32D9, F.Cu at (46.0, 57.5)
- added kibuzzard-68DE34D2: G***, kibuzzard-68DE34D2, F.Cu at (55.5, 50.8)
- added kibuzzard-68DE34F0: G***, kibuzzard-68DE34F0, F.Cu at (85.4, 49.3)
- added kibuzzard-68DE3B40: G***, kibuzzard-68DE3B40, B.Cu at (75.1, 47.4)
- added kibuzzard-68DE3B62: G***, kibuzzard-68DE3B62, B.Cu at (85.3, 48.6)
- added kibuzzard-68DE3EFF: G***, kibuzzard-68DE3EFF, F.Cu at (61.2, 104.9)
- added kibuzzard-68DE3EFF: G***, kibuzzard-68DE3EFF, F.Cu at (61.5, 119.4)
- added kibuzzard-68DE3F2A: G***, kibuzzard-68DE3F2A, B.Cu at (63.0, 53.8)
- added kibuzzard-68DE3F7A: G***, kibuzzard-68DE3F7A, B.Cu at (61.2, 53.8)
- added kibuzzard-68DE3FB0: G***, kibuzzard-68DE3FB0, B.Cu at (86.1, 59.2)
- added kibuzzard-68DFB9FB: G***, kibuzzard-68DFB9FB, B.Cu at (79.9, 98.0)
- added kibuzzard-68DFC30B: G***, kibuzzard-68DFC30B, B.Cu at (43.6, 82.2)
- added kibuzzard-68DFC358: G***, kibuzzard-68DFC358, B.Cu at (43.6, 85.0)
- added kibuzzard-68DFC368: G***, kibuzzard-68DFC368, B.Cu at (43.5, 87.8)
- added kibuzzard-68DFC668: G***, kibuzzard-68DFC668, F.Cu at (48.5, 92.5)
- added kibuzzard-68DFC668: G***, kibuzzard-68DFC668, F.Cu at (83.6, 92.5)
- added kibuzzard-68DFC668: G***, kibuzzard-68DFC668, B.Cu at (83.6, 93.0)
- added kibuzzard-68DFC668: G***, kibuzzard-68DFC668, B.Cu at (75.7, 60.5)
- added kibuzzard-68DFC668: G***, kibuzzard-68DFC668, B.Cu at (48.5, 93.0)
- added kibuzzard-68DFC668: G***, kibuzzard-68DFC668, B.Cu at (58.2, 47.5)
- added kibuzzard-68DFC67B: G***, kibuzzard-68DFC67B, F.Cu at (51.1, 92.5)
- added kibuzzard-68DFC67B: G***, kibuzzard-68DFC67B, F.Cu at (81.0, 92.5)
- added kibuzzard-68DFC67B: G***, kibuzzard-68DFC67B, B.Cu at (58.2, 43.4)
- added kibuzzard-68DFC67B: G***, kibuzzard-68DFC67B, B.Cu at (81.1, 93.0)
- added kibuzzard-68DFC67B: G***, kibuzzard-68DFC67B, B.Cu at (51.1, 93.0)
- added kibuzzard-68DFC69F: G***, kibuzzard-68DFC69F, F.Cu at (78.5, 92.5)
- added kibuzzard-68DFC69F: G***, kibuzzard-68DFC69F, B.Cu at (78.5, 92.9)
- added kibuzzard-68DFC6BF: G***, kibuzzard-68DFC6BF, F.Cu at (53.6, 92.5)
- added kibuzzard-68DFC6BF: G***, kibuzzard-68DFC6BF, B.Cu at (53.6, 93.0)
- added kibuzzard-68DFC753: G***, kibuzzard-68DFC753, B.Cu at (44.5, 114.3)
- added kibuzzard-68DFC753: G***, kibuzzard-68DFC753, B.Cu at (52.1, 106.4)
- added kibuzzard-68DFC753: G***, kibuzzard-68DFC753, B.Cu at (85.9, 111.5)
- added kibuzzard-68DFC753: G***, kibuzzard-68DFC753, B.Cu at (84.8, 114.3)
- added kibuzzard-68DFC76E: G***, kibuzzard-68DFC76E, B.Cu at (58.9, 118.6)
- added kibuzzard-68DFC76E: G***, kibuzzard-68DFC76E, B.Cu at (80.0, 111.0)
- added kibuzzard-68DFC76E: G***, kibuzzard-68DFC76E, B.Cu at (52.1, 119.1)
- added kibuzzard-68DFC76E: G***, kibuzzard-68DFC76E, B.Cu at (87.4, 114.8)
- added kibuzzard-68DFC76E: G***, kibuzzard-68DFC76E, B.Cu at (46.0, 111.3)
- added kibuzzard-68DFC7B6: G***, kibuzzard-68DFC7B6, B.Cu at (82.5, 114.6)
- added kibuzzard-68DFC7C5: G***, kibuzzard-68DFC7C5, B.Cu at (80.0, 114.6)
- added kibuzzard-68DFC824: G***, kibuzzard-68DFC824, B.Cu at (47.0, 119.4)
- added kibuzzard-68DFC82C: G***, kibuzzard-68DFC82C, B.Cu at (49.5, 119.5)
- added kibuzzard-68DFC8BC: G***, kibuzzard-68DFC8BC, B.Cu at (54.1, 106.7)
- added kibuzzard-68DFC8C9: G***, kibuzzard-68DFC8C9, B.Cu at (43.9, 111.3)
- added kibuzzard-68DFC8E0: G***, kibuzzard-68DFC8E0, B.Cu at (48.0, 106.9)
- added kibuzzard-68DFC8EC: G***, kibuzzard-68DFC8EC, B.Cu at (50.0, 107.0)
- added kibuzzard-68DFC952: G***, kibuzzard-68DFC952, B.Cu at (84.1, 111.3)
- added kibuzzard-68DFC958: G***, kibuzzard-68DFC958, B.Cu at (82.0, 111.2)
- added kibuzzard-68DFC96B: G***, kibuzzard-68DFC96B, B.Cu at (78.2, 111.3)
- added kibuzzard-68DFC975: G***, kibuzzard-68DFC975, B.Cu at (88.1, 111.3)
- added kibuzzard-68DFCAC3: G***, kibuzzard-68DFCAC3, B.Cu at (73.2, 60.7)
- added kibuzzard-68DFCACF: G***, kibuzzard-68DFCACF, B.Cu at (70.6, 60.5)
- added kibuzzard-68DFCAE5: G***, kibuzzard-68DFCAE5, B.Cu at (65.5, 60.5)
- added kibuzzard-68DFCAF3: G***, kibuzzard-68DFCAF3, B.Cu at (68.1, 60.5)
- added kibuzzard-68DFCD94: G***, kibuzzard-68DFCD94, F.Cu at (70.4, 65.0)
- added kibuzzard-68DFCDC8: G***, kibuzzard-68DFCDC8, B.Cu at (73.2, 57.9)
- added kibuzzard-68DFCE16: G***, kibuzzard-68DFCE16, F.Cu at (44.6, 57.7)
- added kibuzzard-68DFCE16: G***, kibuzzard-68DFCE16, B.Cu at (44.5, 57.7)
- added kibuzzard-68DFDF18: G***, kibuzzard-68DFDF18, B.Cu at (66.1, 71.8)
- added kibuzzard-68DFE0FD: G***, kibuzzard-68DFE0FD, B.Cu at (64.0, 118.6)
- added kibuzzard-68DFE7B4: G***, kibuzzard-68DFE7B4, B.Cu at (58.3, 45.5)
- D8: footprint LED_SMD:LED_SK6812MINI_PLCC4_3.5x3.5mm_P1.75mm -> CustomLibrary:IN-PI33TBTPRPGPB
- SW2: value SW_DIP_x01 -> SW_gliss; footprint Connector_JST:JST_XH_B2B-XH-A_1x02_P2.50mm_Vertical -> Button_Switch_THT:SW_CK_JS202011AQN_DPDT_Angled; moved to B.Cu
- SW3: footprint TerminalBlock:TerminalBlock_bornier-2_P5.08mm -> Connector_JST:JST_XH_B2B-XH-A_1x02_P2.50mm_Vertical; moved to F.Cu
- moved SW3 12.4 mm to (70.2, 57.8)
- moved J5 10.2 mm to (75.7, 62.6), turned to -90 degrees
- moved R17 9.19 mm to (74.0, 49.0)
- moved R16 9.05 mm to (78.0, 49.0)
- moved J4 5.02 mm to (58.9, 116.6), turned to 0 degrees
- moved R1 3.79 mm to (68.6, 66.0)
- moved SW2 1.82 mm to (72.6, 45.6)
- moved F1 0.85 mm to (69.3, 53.8)
- moved C6 0.66 mm to (76.7, 65.0)
- moved C5 0.31 mm to (88.1, 50.2)
- moved R14 0.30 mm to (83.6, 50.2)
- moved D8 0.28 mm to (52.7, 45.1), turned to 90 degrees
Connections:
- J5 pad 1: TX0 -> GND
- J5 pad 2: RX0 -> EN
- J5 pad 4: EN -> RX0
- J5 pad 5: GND -> TX0
- Q1 pad 1: Net-(J4-Pin_2) -> Net-(J4-Pin_1)
- SW3 pad 2: Net-(J4-Pin_1) -> Net-(J4-Pin_2)
Routing:
- net Net-(J4-Pin_1): track 99.5 -> 16.1 mm, vias 0 -> 1
- net Net-(J4-Pin_2): track 16.1 -> 98.9 mm, vias 1 -> 0
- net GND: track 13.9 -> 23.9 mm, vias 2 -> 255
- net +BATT: track 93.6 -> 101.5 mm
- net EN: track 37.6 -> 45.3 mm, vias 3 -> 4
- net LEVEL_BATTERY: track 33.3 -> 38.5 mm, vias 2 -> 3
- net Net-(D8-DIN): track 10.7 -> 15.0 mm, vias 0 -> 2
- net Net-(SW3-A): track 61.8 -> 58.3 mm
- net +3.3V: track 222.0 -> 225.3 mm, vias 5 -> 3
- net button_user: track 46.0 -> 48.4 mm
- net +5V: track 161.1 -> 159.4 mm, vias 9 -> 8
- net Net-(D1-A): track 33.2 -> 34.2 mm
- net sw_team: track 42.2 -> 42.9 mm
- net RX0: track 16.7 -> 16.0 mm
- net Net-(D8-DOUT): track 5.27 -> 5.38 mm, vias 0 -> 1
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Other:
- outline, holes or cut-outs redrawn
- board text added: ":3"
- board text added: "Bottoms Tops ! We all hate cops!"
- board text added: "Encore un driver de cramé..."
- board text added: "I2C Pullup resistor| v"
- board text added: "Impostor"
- board text added: "Miaou"
- board text added: "PAMIS V1 2026"
- board text added: "This duck is happy"
- board text added: "Wouaf wouaf"
- board text added: "vroom"
