File: kicad_pami/pami_2026/_autosave-pami_2026.kicad_pcb (KiCad board)
At the start: 4 copper layers, 50 x 80 mm, 69 parts, among them J1 Conn_01x04_Socket, J10 Conn_01x07_Socket, J11 Conn_01x06, J12 Conn_01x06, J14 Conn_01x03_Pin, J2 Conn_01x03_Pin, J3 Conn_01x04_Pin, J4 Conn_01x02_Pin, J5 Conn_01x05_Pin, J7 Conn_01x03_Pin, J8 USB_C_Receptacle_USB2.0_14P, J9 Conn_01x04_Pin, Q1 NMOS, Q2 NMOS, Q3 NMOS, SW1 SW_Push, SW2 SW_DIP_x01, SW3 SW_Push_Open, SW4 SW_Reed, SW5 SW_Push, SW6 SW_Push, U1 DRV8833RTY, U2 ESP32-S3-MINI-1, U3 LD1117S33TR_SOT223, U4 L7805

Commit message: V0.2 cad
Parts:
- SW2: footprint Connector_JST:JST_XH_B2B-XH-A_1x02_P2.50mm_Vertical -> Button_Switch_THT:SW_CK_JS202011AQN_DPDT_Angled
- moved SW2 3.97 mm to (77.7, 45.8), turned to 180 degrees
Routing:
- net EN: track 37.6 -> 43.4 mm
- net sw_team: track 42.2 -> 38.2 mm
