File: kicad_pami/pami_2026/pami_2026.kicad_sch (KiCad schematic)
At the start: 12 parts, among them J3 Conn_01x04_Pin, J8 USB_C_Receptacle_USB2.0_14P, J9 Conn_01x04_Pin, SW1 SW_Push, SW2 SW_DIP_x01, SW4 SW_Reed, U2 ESP32-S3-MINI-1

Commit message: ajout code / avancement pcb et 3D
Parts:
- added C5, C6, C7: 100n, Capacitor_SMD:C_0805_2012Metric_Pad1.18x1.45mm_HandSolder, symbol Device:C
- added D1: D, Diode_SMD:D_0805_2012Metric, symbol Device:D
- added J5: Conn_01x05_Pin, Connector_PinHeader_2.54mm:PinHeader_1x05_P2.54mm_Vertical, symbol Connector:Conn_01x05_Pin
- added R14: R, Resistor_SMD:R_0805_2012Metric_Pad1.20x1.40mm_HandSolder, symbol Device:R
- added SW5, SW6: SW_Push, CustomLibrary:PTS645VSM19PSMTR92LFS, symbol Switch:SW_Push
- J8: footprint Connector_USB:USB_C_Receptacle_GCT_USB4105-xx-A_16P_TopMnt_Horizontal -> CustomLibrary:MOLEX_2169890001
- SW1: footprint Button_Switch_THT:SW_Tactile_SPST_Angled_PTS645Vx39-2LFS -> Button_Switch_SMD:SW_Push_1P1T_NO_CK_KSC9xxJ
- U2: footprint RF_Module:ESP32-S2-MINI-1 -> CustomLibrary:ESP32S3MINI1N8
Connections:
- net +3.3V: now also R14.1
- net GND: now also C5.2, C6.2, C7.2, J5.5 (Pin_5), SW5.2, SW6.1
- net I2C_scl: now also U2.20 (IO16)
- net I2C_sda: now also U2.21 (IO17)
- net LEVEL_BATTERY: now also U2.19 (IO15)
- net NEOPIXEL: now also U2.29 (IO34)
- net RX_lidar: now also U2.25 (IO21)
- net SERVO1: now also U2.13 (IO9)
- net SERVO2: now also U2.12 (IO8)
- net TX_lidar: now also U2.26 (IO26)
- net motor_a+: now also U2.15 (IO11)
- net motor_a-: now also U2.16 (IO12)
- net motor_a_sense: now also U2.9 (IO5)
- net motor_b+: now also U2.17 (IO13)
- net motor_b-: now also U2.18 (IO14)
- net motor_b_sense: now also U2.10 (IO6)
- net motor_enable: now also U2.14 (IO10)
- net motor_enc_a+: now also U2.8 (IO4)
- net motor_enc_a-: now also U2.7 (IO3)
- net motor_enc_b+: now also U2.6 (IO2)
- net motor_enc_b-: now also U2.5 (IO1)
- net motor_fault: now also U2.11 (IO7)
- net sw_team: now also U2.27 (IO47)
- net sw_tirette: now also U2.30 (IO48)
- net tft_cs: now also U2.35 (IO39)
- net tft_dc: now also U2.33 (IO37)
- net tft_rst: now also U2.34 (IO38)
- net tft_scl: now also U2.32 (IO36)
- net EN: now reaches R1.2, SW1.2, U2.45 (EN)
- net EN: now also C6.1, J5.4 (Pin_4)
- net at J8.A4 (VBUS), J8.A9 (VBUS), J8.B4 (VBUS)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: now also D1.2 (A)
- net EN_SCREEN: now reaches U2.22 (IO18)
- net button_user: now reaches U2.28 (IO33)
- net button_user: now also C7.1, SW6.2
- net tft_sda: now reaches U2.31 (IO35)
- net TX0: now reaches U2.39 (TXD0)
- net TX0: now also J5.1 (Pin_1)
- net GPIO0: now reaches U2.4 (IO0)
- net GPIO0: now also C5.1, J5.3 (Pin_3), R14.2, SW5.1
- net RX0: now reaches U2.40 (RXD0)
- net RX0: now also J5.2 (Pin_2)
- new net +5V: D1.1 (K)
- no-connect marks 0 -> 2
Other:
- note added: "ADC1_4 ADC1_5"
- note added: "ADC1_9"
- note added: "GPIO 45 BOOT PIN GPIO 46 BOOT PIN"
- note added: "GPIO0 BOOT PIN"
- note added: "Optionnal | Error <--| Motor |"
- note added: "the ADC2 is shared with the WIFI module cannot be used simultaneoustly"

Commit message: fin PCB
Parts:
- SW2: value SW_DIP_x01 -> SW_gliss; footprint Connector_JST:JST_XH_B2B-XH-A_1x02_P2.50mm_Vertical -> Button_Switch_THT:SW_CK_JS202011AQN_DPDT_Angled
Connections:
- net EN: now also J5.2 (Pin_2); no longer J5.4 (Pin_4)
- net GND: now also J5.1 (Pin_1); no longer J5.5 (Pin_5)
- net RX0: now also J5.4 (Pin_4); no longer J5.2 (Pin_2)
- net TX0: now also J5.5 (Pin_5); no longer J5.1 (Pin_1)
Changed lines of the file:
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@@
 			)
 		)
-		(property "Value" "SW_DIP_x01"
+		(property "Value" "SW_gliss"
 			(at 266.7 30.48 0)
 			(effects
@@
 			)
 		)
-		(property "Footprint" "Connector_JST:JST_XH_B2B-XH-A_1x02_P2.50mm_Vertical"
+		(property "Footprint" "Button_Switch_THT:SW_CK_JS202011AQN_DPDT_Angled"
 			(at 266.7 35.56 0)
 			(effects
@@
 		(lib_id "Connector:Conn_01x05_Pin")
 		(at 170.18 132.08 0)
+		(mirror x)
 		(unit 1)
 		(exclude_from_sim no)
@@
 		(on_board yes)
 		(dnp no)
-		(fields_autoplaced yes)
 		(property "Reference" "J5"
-			(at 170.815 121.92 0)
+			(at 170.815 142.24 0)
 			(effects
 				(font
@@
 		)
 		(property "Value" "Conn_01x05_Pin"
-			(at 170.815 124.46 0)
+			(at 170.815 139.7 0)
 			(effects
 				(font
